Commit message: comment out vision odom tf and topics in order to maintain the tf tree of lvi-sam

File: spot_description/urdf/spot.urdf.xacro (robot description, xacro)
@@ -13,10 +13,17 @@
         </collision>
     </link>
-    <link name="base_link"/>
+    <!-- <link name="map"/> -->
+    <!-- <link name="odom"/>
+    <joint name="odom_map" type="fixed">
+        <origin xyz="0 0 0" rpy="0 0 0" />
+        <parent link="map" />
+        <child link="odom" />
+    </joint> -->
+    <!-- <link name="base_link"/>
     <joint name="base_link_joint" type="fixed">
         <origin xyz="0 0 0" rpy="0 0 0" />
         <parent link="body" />
         <child link="base_link" />
-    </joint>
+    </joint> -->
     <link name="front_rail"/>
     <joint name="front_rail_joint" type="fixed">
@@ -260,4 +267,5 @@
     </joint>
     <link name="ouster_link"/>
+    <!-- <link name="lidar_link"/> -->
     <link name ="imu_link"/>
     <joint name="ouster_joint" type="fixed">
@@ -266,4 +274,9 @@
         <child link="ouster_link" />
     </joint>
+    <!-- <joint name="ouster_lvisam" type="fixed">
+        <origin xyz="0 0 -0.31" rpy="0 0 0" />
+        <parent link="lidar_link" />
+        <child link="body" />
+    </joint> -->
     <joint name="ouster_imu_joint" type="fixed">
         <origin xyz="-0.157242 -0.061091 -0.020754" rpy="-3.1415926 0 0" />

Commit message: add imu link

File: spot_description/urdf/spot.urdf.xacro (robot description, xacro)
@@ -260,8 +260,14 @@
     </joint>
     <link name="ouster_link"/>
+    <link name ="imu_link"/>
     <joint name="ouster_joint" type="fixed">
-        <origin xyz="0 0 0.31" rpy="0 0 3.141" />
+        <origin xyz="0 0 0.31" rpy="0 0 0" />
         <parent link="body" />
         <child link="ouster_link" />
+    </joint>
+    <joint name="ouster_imu_joint" type="fixed">
+        <origin xyz="-0.157242 -0.061091 -0.020754" rpy="-3.1415926 0 0" />
+        <parent link="ouster_link" />
+        <child link="imu_link" />
     </joint>
     <!-- Standard accessories. -->

Commit message: adapt to mist spot

File: spot_description/urdf/spot.urdf.xacro (robot description, xacro)
@@ -258,4 +258,10 @@
         <child link="rear_right_lower_leg" />
         <limit effort="1000" velocity="1000.00" lower="-2.7929" upper="-0.257725" />
+    </joint>
+    <link name="ouster_link"/>
+    <joint name="ouster_joint" type="fixed">
+        <origin xyz="0 0 0.31" rpy="0 0 3.141" />
+        <parent link="body" />
+        <child link="ouster_link" />
     </joint>
     <!-- Standard accessories. -->
